File: power.kicad_sch (KiCad schematic)
At the start: 7 parts, among them U1 AP2114HA-3.3TRG1

Commit message: Add servo connectors
Parts:
- removed C8, C9: 4.7u, Capacitor_SMD:C_0805_2012Metric_Pad1.18x1.45mm_HandSolder, symbol Device:C
- removed D1, D4: LED, LED_SMD:LED_0805_2012Metric_Pad1.15x1.40mm_HandSolder, symbol Device:LED
- removed R1, R10: 1k, Resistor_SMD:R_0402_1005Metric_Pad0.72x0.64mm_HandSolder, symbol Device:R
- removed U1: AP2114HA-3.3TRG1, Package_TO_SOT_SMD:SOT-223-3_TabPin2, symbol mc_custom_symbols:AP2114H-3.3TRG1
Other:
- note removed: "Voltage Regulator"
