File: mcu.kicad_sch (KiCad schematic)
At the start: 24 parts, among them J2 Conn_01x05_Pin, SW1 SW_Push, SW2 SW_Push, SW3 SW_Push, U2 STM32H503CBTx, Y1 CX3225FB16000F0FZZH1 16MHz

Commit message: Update schematic
Connections:
- net NRST: now also J2.5 (Pin_5)
- net SWCLK: now also J2.4 (Pin_4)
- net SWDIO: now also J2.3 (Pin_3)
- net PA1 renamed UART1_RX
- net PA2 renamed UART1_TX
- net PB5 renamed I2C_SDA
- net PB6 renamed I2C_SCL
