File: usb_c.kicad_sch (KiCad schematic)
At the start: 19 parts, among them J1 USB_C_Receptacle_USB2.0_16P, U1 AP2114HA-3.3TRG1, U3 USBLC6-2SC6, U4 CP2102N-Axx-xQFN20

Commit message: Update schematic
Parts:
- added R14: 10k, symbol Device:R
- R6: value R -> 1k
Connections:
- net GND: now also R14.2
- net at U4.11 (~{SUSPEND}): now also R14.1
- net RX renamed CP2102_RX
- net TX renamed CP2102_TX
- no-connect marks 2 -> 10
Other:
- note removed: "Have to check it with waveshare board"
Changed lines of the file:
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@@
 		)
 	)
-	(text "Have to check it with waveshare board"
-		(exclude_from_sim no)
-		(at 115.062 80.518 0)
-		(effects
-			(font
-				(size 1.27 1.27)
-			)
-		)
-	)
 	(text "Voltage Regulator\nVBUS -> 3V3"
 		(exclude_from_sim no)
-		(at 82.55 143.002 0)
+		(at 82.296 141.732 0)
 		(effects
 			(font
@@
 	)
 	(no_connect
+		(at 91.44 90.17)
+	)
+	(no_connect
+		(at 91.44 64.77)
+	)
+	(no_connect
 		(at 223.52 88.9)
 	)
 	(no_connect
+		(at 91.44 92.71)
+	)
+	(no_connect
+		(at 91.44 95.25)
+	)
+	(no_connect
 		(at 223.52 91.44)
 	)
+	(no_connect
+		(at 91.44 97.79)
+	)
+	(no_connect
+		(at 91.44 82.55)
+	)
+	(no_connect
+		(at 91.44 67.31)
+	)
+	(no_connect
+		(at 91.44 74.93)
+	)
 	(wire
 		(pts
@@
 	(polyline
 		(pts
-			(xy 12.7 134.62) (xy 153.67 134.62)
+			(xy 12.7 133.35) (xy 153.67 133.35)
 		)
 		(stroke
@@
 	(wire
 		(pts
+			(xy 91.44 85.09) (xy 99.06 85.09)
+		)
+		(stroke
+			(width 0)
+			(type default)
+		)
+	)
+	(wire
+		(pts
 			(xy 209.55 91.44) (xy 213.36 91.44)
 		)
@@
 	(wire
 		(pts
+			(xy 99.06 85.09) (xy 99.06 87.63)
+		)
+		(stroke
+			(width 0)
+			(type default)
+		)
+	)
+	(wire
+		(pts
 			(xy 96.52 168.91) (xy 101.6 168.91)
 		)
@@
 	(wire
 		(pts
+			(xy 99.06 95.25) (xy 99.06 97.79)
+		)
+		(stroke
+			(width 0)
+			(type default)
+		)
+	)
+	(wire
+		(pts
 			(xy 189.23 91.44) (xy 199.39 91.44)
 		)
@@
 		)
 	)
-	(hierarchical_label "TX"
+	(hierarchical_label "CP2102_TX"
 		(shape output)
 		(at 95.25 59.69 0)
@@
 		)
 	)
-	(hierarchical_label "RX"
+	(hierarchical_label "CP2102_RX"
 		(shape input)
 		(at 95.25 62.23 0)
@@
 			)
 		)
-		(property "Value" "R"
+		(property "Value" "1k"
 			(at 66.04 54.6099 0)
 			(show_name no)
@@
 	)
 	(symbol
+		(lib_id "Device:R")
+		(at 99.06 91.44 0)
+		(unit 1)
+		(body_style 1)
+		(exclude_from_sim no)
+		(in_bom yes)
+		(on_board yes)
+		(in_pos_files yes)
+		(dnp no)
+		(fields_autoplaced yes)
+		(property "Reference" "R14"
+			(at 101.6 90.1699 0)
+			(show_name no)
+			(do_not_autoplace no)
+			(effects
+				(font
+					(size 1.27 1.27)
+				)
+				(justify left)
+			)
+		)
+		(property "Value" "10k"
+			(at 101.6 92.7099 0)
+			(show_name no)
+			(do_not_autoplace no)
+			(effects
+				(font
+					(size 1.27 1.27)
+				)
+				(justify left)
+			)
+		)
+		(property "Footprint" ""
+			(at 97.282 91.44 90)
+			(hide yes)
+			(show_name no)
+			(do_not_autoplace no)
+			(effects
+				(font
+					(size 1.27 1.27)
+				)
+			)
+		)
+		(property "Datasheet" ""
+			(at 99.06 91.44 0)
+			(hide yes)
+			(show_name no)
+			(do_not_autoplace no)
+			(effects
+				(font
+					(size 1.27 1.27)
+				)
+			)
+		)
+		(property "Description" "Resistor"
+			(at 99.06 91.44 0)
+			(hide yes)
+			(show_name no)
+			(do_not_autoplace no)
+			(effects
+				(font
+					(size 1.27 1.27)
+				)
+			)
+		)
+		(pin "2"
+		)
+		(pin "1"
+		)
+		(instances
+			(project "pisarz-mainboard"
+				(path "/3fa3a621-8f50-4a33-bd41-24b098d8d0ef/5eae9f20-c0db-468d-b61d-7762ef488b79"
+					(reference "R14")
+					(unit 1)
+				)
+			)
+		)
+	)
+	(symbol
 		(lib_id "power:GND")
 		(at 82.55 180.34 0)
@@
 					(unit 1)
 				)
+			)
+		)
+	)
+	(symbol
+		(lib_id "power:GND")
+		(at 99.06 97.79 0)
+		(unit 1)
+		(body_style 1)
+		(exclude_from_sim no)
+		(in_bom yes)
+		(on_board yes)
+		(in_pos_files yes)
+		(dnp no)
+		(fields_autoplaced yes)
+		(property "Reference" "#PWR049"
+			(at 99.06 104.14 0)
+			(hide yes)
+			(show_name no)
+			(do_not_autoplace no)
+			(effects
+				(font
+					(size 1.27 1.27)
+				)
+			)
+		)
+		(property "Value" "GND"
+			(at 99.06 102.87 0)
+			(show_name no)
+			(do_not_autoplace no)
+			(effects
+				(font
+					(size 1.27 1.27)
+				)
+			)
+		)
+		(property "Footprint" ""
+			(at 99.06 97.79 0)
+			(hide yes)
+			(show_name no)
+			(do_not_autoplace no)
+			(effects
+				(font
+					(size 1.27 1.27)
+				)
+			)
+		)
+		(property "Datasheet" ""
+			(at 99.06 97.79 0)
+			(hide yes)
+			(show_name no)
+			(do_not_autoplace no)
+			(effects
+				(font
+					(size 1.27 1.27)
+				)
+			)
+		)
+		(property "Description" "Power symbol creates a global label with name \"GND\" , ground"
+			(at 99.06 97.79 0)
+			(hide yes)
+			(show_name no)
+			(do_not_autoplace no)
+			(effects
+				(font
+					(size 1.27 1.27)
+				)
+			)
+		)
+		(pin "1"
+		)
+		(instances
+			(project "pisarz-mainboard"
+				(path "/3fa3a621-8f50-4a33-bd41-24b098d8d0ef/5eae9f20-c0db-468d-b61d-7762ef488b79"
+					(reference "#PWR049")
+					(unit 1)
+				)
